File: KiCAD/Circuit Board/Circuit Board.sch (KiCad schematic (older format))
At the start: 9 parts

Commit message: Designed circuit. Should work
Parts:
- added SW?: SW_DIP_x01, symbol Switch:SW_DIP_x01
Connections:
- net +9V: now also SW?.1; no longer J?.4 (Pin_4), U?.15 (VIN)
- new net +9VA: J?.4 (Pin_4), SW?.2
Changed lines of the file:
@@
 	1    0    0    -1
-$EndComp
-$Comp
-L power:+9V #PWR?
-U 1 1 5FB79B0C
-P 8050 2850
-F 0 "#PWR?" H 8050 2700 50  0001 C CNN
-F 1 "+9V" V 8065 2978 50  0000 L CNN
-F 2 "" H 8050 2850 50  0001 C CNN
-F 3 "" H 8050 2850 50  0001 C CNN
-	1    8050 2850
-	0    -1   -1   0
 $EndComp
 Text GLabel 6800 1550 1    50   Input ~ 0
@@
 	0    1    1    0
 $EndComp
-$Comp
-L power:+9V #PWR?
-U 1 1 5FB87969
-P 2800 3400
-F 0 "#PWR?" H 2800 3250 50  0001 C CNN
-F 1 "+9V" V 2815 3528 50  0000 L CNN
-F 2 "" H 2800 3400 50  0001 C CNN
-F 3 "" H 2800 3400 50  0001 C CNN
-	1    2800 3400
-	0    -1   -1   0
-$EndComp
 Text GLabel 4400 2400 2    50   Input ~ 0
 D4-R-Sw
@@
 Text GLabel 6200 1750 0    50   Input ~ 0
 Sw-R
+$Comp
+L Switch:SW_DIP_x01 SW?
+U 1 1 5FB8FACD
+P 1850 3400
+F 0 "SW?" H 1850 3667 50  0000 C CNN
+F 1 "SW_DIP_x01" H 1850 3576 50  0000 C CNN
+F 2 "" H 1850 3400 50  0001 C CNN
+F 3 "~" H 1850 3400 50  0001 C CNN
+	1    1850 3400
+	1    0    0    -1
+$EndComp
+$Comp
+L power:+9V #PWR?
+U 1 1 5FB911D2
+P 1550 3400
+F 0 "#PWR?" H 1550 3250 50  0001 C CNN
+F 1 "+9V" V 1565 3528 50  0000 L CNN
+F 2 "" H 1550 3400 50  0001 C CNN
+F 3 "" H 1550 3400 50  0001 C CNN
+	1    1550 3400
+	0    -1   -1   0
+$EndComp
+$Comp
+L power:+9VA #PWR?
+U 1 1 5FB91FE5
+P 2150 3400
+F 0 "#PWR?" H 2150 3275 50  0001 C CNN
+F 1 "+9VA" V 2165 3528 50  0000 L CNN
+F 2 "" H 2150 3400 50  0001 C CNN
+F 3 "" H 2150 3400 50  0001 C CNN
+	1    2150 3400
+	0    1    1    0
+$EndComp
+$Comp
+L power:+9VA #PWR?
+U 1 1 5FB921DC
+P 8050 2850
+F 0 "#PWR?" H 8050 2725 50  0001 C CNN
+F 1 "+9VA" V 8065 2977 50  0000 L CNN
+F 2 "" H 8050 2850 50  0001 C CNN
+F 3 "" H 8050 2850 50  0001 C CNN
+	1    8050 2850
+	0    -1   -1   0
+$EndComp
 $EndSCHEMATC

Commit message: hothing of interest
Parts:
- J1: renamed from J?; footprint (none) -> Pin_Headers:Pin_Header_Angled_1x04_Pitch2.54mm
- R1, R2, R3: renamed from R?; footprint (none) -> Resistors_ThroughHole:R_Axial_DIN0411_L9.9mm_D3.6mm_P7.62mm_Vertical
- gave numbers to parts that had none: 6
Changed lines of the file:
@@
 $EndDescr
 $Comp
-L Transistor_BJT:BD437 Q?
+L Transistor_BJT:BD437 Q1
 U 1 1 5FB6EE4D
 P 6700 1750
-F 0 "Q?" H 6892 1796 50  0000 L CNN
+F 0 "Q1" H 6892 1796 50  0000 L CNN
 F 1 "BD437" H 6892 1705 50  0000 L CNN
 F 2 "Package_TO_SOT_THT:TO-126-3_Vertical" H 6900 1675 50  0001 L CIN
@@
 $EndComp
 $Comp
-L Transistor_BJT:BD437 Q?
+L Transistor_BJT:BD437 Q2
 U 1 1 5FB711C4
 P 6700 2700
-F 0 "Q?" H 6892 2746 50  0000 L CNN
+F 0 "Q2" H 6892 2746 50  0000 L CNN
 F 1 "BD437" H 6892 2655 50  0000 L CNN
 F 2 "Package_TO_SOT_THT:TO-126-3_Vertical" H 6900 2625 50  0001 L CIN
@@
 $EndComp
 $Comp
-L Transistor_BJT:BD437 Q?
+L Transistor_BJT:BD437 Q3
 U 1 1 5FB726F4
 P 6700 3700
-F 0 "Q?" H 6892 3746 50  0000 L CNN
+F 0 "Q3" H 6892 3746 50  0000 L CNN
 F 1 "BD437" H 6892 3655 50  0000 L CNN
 F 2 "Package_TO_SOT_THT:TO-126-3_Vertical" H 6900 3625 50  0001 L CIN
@@
 B_LED
 $Comp
-L Connector_Generic:Conn_01x04 J?
+L Connector_Generic:Conn_01x04 J1
 U 1 1 5FB77CA4
 P 8250 2650
-F 0 "J?" H 8330 2642 50  0000 L CNN
+F 0 "J1" H 8330 2642 50  0000 L CNN
 F 1 "Conn_01x04" H 8330 2551 50  0000 L CNN
-F 2 "" H 8250 2650 50  0001 C CNN
+F 2 "Pin_Headers:Pin_Header_Angled_1x04_Pitch2.54mm" H 8250 2650 50  0001 C CNN
 F 3 "~" H 8250 2650 50  0001 C CNN
 	1    8250 2650
@@
 B_LED
 $Comp
-L power:GND #PWR?
+L power:GND #PWR0101
 U 1 1 5FB7DFA5
 P 6800 2900
-F 0 "#PWR?" H 6800 2650 50  0001 C CNN
+F 0 "#PWR0101" H 6800 2650 50  0001 C CNN
 F 1 "GND" H 6805 2727 50  0000 C CNN
 F 2 "" H 6800 2900 50  0001 C CNN
@@
 $EndComp
 $Comp
-L power:GND #PWR?
+L power:GND #PWR0102
 U 1 1 5FB7EB81
 P 6800 1950
-F 0 "#PWR?" H 6800 1700 50  0001 C CNN
+F 0 "#PWR0102" H 6800 1700 50  0001 C CNN
 F 1 "GND" H 6805 1777 50  0000 C CNN
 F 2 "" H 6800 1950 50  0001 C CNN
@@
 $EndComp
 $Comp
-L power:GND #PWR?
+L power:GND #PWR0103
 U 1 1 5FB7F30B
 P 6800 3900
-F 0 "#PWR?" H 6800 3650 50  0001 C CNN
+F 0 "#PWR0103" H 6800 3650 50  0001 C CNN
 F 1 "GND" H 6805 3727 50  0000 C CNN
 F 2 "" H 6800 3900 50  0001 C CNN
@@
 $EndComp
 $Comp
-L Device:R R?
+L Device:R R2
 U 1 1 5FB80264
 P 6350 2700
-F 0 "R?" V 6143 2700 50  0000 C CNN
+F 0 "R2" V 6143 2700 50  0000 C CNN
 F 1 "1500" V 6234 2700 50  0000 C CNN
-F 2 "" V 6280 2700 50  0001 C CNN
+F 2 "Resistors_ThroughHole:R_Axial_DIN0411_L9.9mm_D3.6mm_P7.62mm_Vertical" V 6280 2700 50  0001 C CNN
 F 3 "~" H 6350 2700 50  0001 C CNN
 	1    6350 2700
@@
 $EndComp
 $Comp
-L Device:R R?
+L Device:R R1
 U 1 1 5FB8173A
 P 6350 1750
-F 0 "R?" V 6143 1750 50  0000 C CNN
+F 0 "R1" V 6143 1750 50  0000 C CNN
 F 1 "1500" V 6234 1750 50  0000 C CNN
-F 2 "" V 6280 1750 50  0001 C CNN
+F 2 "Resistors_ThroughHole:R_Axial_DIN0411_L9.9mm_D3.6mm_P7.62mm_Vertical" V 6280 1750 50  0001 C CNN
 F 3 "~" H 6350 1750 50  0001 C CNN
 	1    6350 1750
@@
 $EndComp
 $Comp
-L Device:R R?
+L Device:R R3
 U 1 1 5FB8241D
 P 6350 3700
-F 0 "R?" V 6143 3700 50  0000 C CNN
+F 0 "R3" V 6143 3700 50  0000 C CNN
 F 1 "1500" V 6234 3700 50  0000 C CNN
-F 2 "" V 6280 3700 50  0001 C CNN
+F 2 "Resistors_ThroughHole:R_Axial_DIN0411_L9.9mm_D3.6mm_P7.62mm_Vertical" V 6280 3700 50  0001 C CNN
 F 3 "~" H 6350 3700 50  0001 C CNN
 	1    6350 3700
@@
 $EndComp
 $Comp
-L power:GND #PWR?
+L power:GND #PWR0104
 U 1 1 5FB865C7
 P 2800 3300
-F 0 "#PWR?" H 2800 3050 50  0001 C CNN
+F 0 "#PWR0104" H 2800 3050 50  0001 C CNN
 F 1 "GND" V 2805 3172 50  0000 R CNN
 F 2 "" H 2800 3300 50  0001 C CNN
@@
 D4-R-Sw
 $Comp
-L ESP8266:NodeMCU_1.0_(ESP-12E) U?
+L ESP8266:NodeMCU_1.0_(ESP-12E) U1
 U 1 1 5FB839C8
 P 3600 2700
-F 0 "U?" H 3600 3787 60  0000 C CNN
+F 0 "U1" H 3600 3787 60  0000 C CNN
 F 1 "NodeMCU_1.0_(ESP-12E)" H 3600 3681 60  0000 C CNN
-F 2 "" H 3000 1850 60  0000 C CNN
+F 2 "" H 3000 1850 60  0001 C CNN
 F 3 "" H 3000 1850 60  0000 C CNN
 	1    3600 2700
@@
 D2-G-Sw
 $Comp
-L Switch:SW_DIP_x03 SW?
+L Switch:SW_DIP_x03 SW2
 U 1 1 5FB89BE0
 P 5350 3250
-F 0 "SW?" H 5350 3717 50  0000 C CNN
+F 0 "SW2" H 5350 3717 50  0000 C CNN
 F 1 "SW_DIP_x03" H 5350 3626 50  0000 C CNN
 F 2 "" H 5350 3250 50  0001 C CNN
@@
 Sw-R
 $Comp
-L Switch:SW_DIP_x01 SW?
+L Switch:SW_DIP_x01 SW1
 U 1 1 5FB8FACD
 P 1850 3400
-F 0 "SW?" H 1850 3667 50  0000 C CNN
+F 0 "SW1" H 1850 3667 50  0000 C CNN
 F 1 "SW_DIP_x01" H 1850 3576 50  0000 C CNN
 F 2 "" H 1850 3400 50  0001 C CNN
@@
 $EndComp
 $Comp
-L power:+9V #PWR?
+L power:+9V #PWR0105
 U 1 1 5FB911D2
 P 1550 3400
-F 0 "#PWR?" H 1550 3250 50  0001 C CNN
+F 0 "#PWR0105" H 1550 3250 50  0001 C CNN
 F 1 "+9V" V 1565 3528 50  0000 L CNN
 F 2 "" H 1550 3400 50  0001 C CNN
@@
 $EndComp
 $Comp
-L power:+9VA #PWR?
+L power:+9VA #PWR0106
 U 1 1 5FB91FE5
 P 2150 3400
-F 0 "#PWR?" H 2150 3275 50  0001 C CNN
+F 0 "#PWR0106" H 2150 3275 50  0001 C CNN
 F 1 "+9VA" V 2165 3528 50  0000 L CNN
 F 2 "" H 2150 3400 50  0001 C CNN
@@
 $EndComp
 $Comp
-L power:+9VA #PWR?
+L power:+9VA #PWR0107
 U 1 1 5FB921DC
 P 8050 2850
-F 0 "#PWR?" H 8050 2725 50  0001 C CNN
+F 0 "#PWR0107" H 8050 2725 50  0001 C CNN
 F 1 "+9VA" V 8065 2977 50  0000 L CNN
 F 2 "" H 8050 2850 50  0001 C CNN
