File: KiCAD/ESP12 Circuit Board/ESP12E Circuit Board/ESP12E Circuit Board.kicad_pcb (KiCad board)
At the start: 2 copper layers, 1 part, among them U1 ESP8266-12E_ESP-12E

Commit message: worked on the smd circuit
Parts:
- added 10uF1: CP, Capacitors_SMD:C_0603_HandSoldering, F.Cu at (157.5, 116.1)
- added 1uF1: CP, Capacitors_SMD:C_0603_HandSoldering, F.Cu at (157.5, 123.2)
- added 470pF1: CP, Capacitors_SMD:C_0603_HandSoldering, F.Cu at (160.3, 119.6)
- added J1: Conn_01x04_Male, Pin_Headers:Pin_Header_Straight_1x04_Pitch2.54mm, F.Cu at (172.0, 109.7)
- added J2: Conn_01x02_Female, Pin_Headers:Pin_Header_Straight_1x02_Pitch2.54mm, F.Cu at (171.7, 121.2)
- added Q1: BCP56, BCP54-16 footprint:SOT230P700X180-4N, F.Cu at (165.4, 112.0)
- added Q2: BCP56, BCP54-16 footprint:SOT230P700X180-4N, F.Cu at (165.4, 120.3)
- added Q3: BCP56, BCP54-16 footprint:SOT230P700X180-4N, F.Cu at (165.4, 104.1)
- added RN1: 1500, Resistors_SMD:R_Array_Concave_4x0603, F.Cu at (159.0, 109.5)
- added U2: SPX3819M5-L-3-3, TO_SOT_Packages_SMD:SOT-23-5_HandSoldering, F.Cu at (157.5, 119.6)
- moved U1 15.8 mm to (146.6, 109.7), turned to 180 degrees
Connections:
- U1 pad 8: Net-(U1-Pad8) -> +3V3
