File: KiCAD/ESP12 Circuit Board Throughole/ESP12E Circuit Board/ESP12E Circuit Board.kicad_pcb (KiCad board)
At the start: 2 copper layers, 13 parts, among them J1 Conn_01x04_Male, J2 Conn_01x02_Female, Q1 BD437, Q2 BD437, Q3 BD437, U1 ESP8266-12E_ESP-12E, U2 SPX3819M5-L-3-3

Commit message: worked on tht circuit
Parts:
- moved J1 24.5 mm to (161.3, 108.7), turned to 270 degrees
- moved U2 17.0 mm to (146.8, 92.5), turned to 90 degrees
- moved Q1 16.8 mm to (154.4, 102.4), turned to 90 degrees
- moved 470pF1 16.1 mm to (149.6, 92.5), turned to 270 degrees
- moved R2 16.0 mm to (160.3, 96.5), turned to 90 degrees
- moved 1uF1 14.7 mm to (146.8, 96.0)
- moved 10uF1 14.2 mm to (146.8, 88.9)
- moved J2 11.2 mm to (148.8, 108.7), turned to 270 degrees
- moved R1 10.1 mm to (156.5, 96.5), turned to 90 degrees
- moved Q2 9.84 mm to (159.0, 102.4), turned to 90 degrees
- moved U1 6.15 mm to (134.9, 97.5), turned to 180 degrees
- moved R3 5.26 mm to (152.9, 96.5), turned to 90 degrees
- moved Q3 2.28 mm to (149.9, 102.4), turned to 90 degrees

Commit message: worked on tht
Parts:
- moved Q3 9.14 mm to (159.0, 102.4)
- moved R3 7.37 mm to (160.3, 96.5)
- moved Q2 4.57 mm to (154.4, 102.4)
- moved Q1 4.57 mm to (149.9, 102.4)
- moved R2 3.81 mm to (156.5, 96.5)
- moved R1 3.56 mm to (152.9, 96.5)
Routing:
- net GND: track 0.00 -> 44.3 mm
- net +9V: track 0.00 -> 36.3 mm
- net B_LED: track 0.00 -> 10.1 mm
- net G_LED: track 0.00 -> 8.72 mm
- net R_LED: track 0.00 -> 8.44 mm
- net +3V3: track 0.00 -> 5.93 mm
- net Net-(Q1-PadB): track 0.00 -> 4.29 mm
- net Net-(Q2-PadB): track 0.00 -> 3.87 mm
- net Net-(Q3-PadB): track 0.00 -> 3.56 mm
- net Net-(470pF1-Pad1): track 0.00 -> 2.01 mm
- added copper zone on B.Cu, net GND
